Commit message: quad

File: body.urdf (robot description, URDF)
Before this commit: robot robot, 3 links, 2 joints
Links:
- added link BackLowerLeg, mass 1; collision box size=0.2 0.2 1; visual box size=0.2 0.2 1
- added link FrontLowerLeg, mass 1; collision box size=0.2 0.2 1; visual box size=0.2 0.2 1
- added link LeftLeg, mass 1; collision box size=1 0.2 0.2; visual box size=1 0.2 0.2
- added link LeftLowerLeg, mass 1; collision box size=0.2 0.2 1; visual box size=0.2 0.2 1
- added link RightLeg, mass 1; collision box size=1 0.2 0.2; visual box size=1 0.2 0.2
- added link RightLowerLeg, mass 1; collision box size=0.2 0.2 1; visual box size=0.2 0.2 1
- link BackLeg: geometry collision box size=0.2 1 0.2; visual box size=0.2 1 0.2
- link FrontLeg: geometry collision box size=0.2 1 0.2; visual box size=0.2 1 0.2
Joints:
- added joint BackLeg_BackLowerLeg: type revolute, parent BackLeg, child BackLowerLeg, origin xyz=0 -1 0 rpy=0 0 0, axis 1 0 0, limit lower=-3.14159 upper=3.14159 effort=0.0 velocity=0.0
- added joint FrontLeg_FrontLowerLeg: type revolute, parent FrontLeg, child FrontLowerLeg, origin xyz=0 1 0 rpy=0 0 0, axis 1 0 0, limit lower=-3.14159 upper=3.14159 effort=0.0 velocity=0.0
- added joint LeftLeg_LeftLowerLeg: type revolute, parent LeftLeg, child LeftLowerLeg, origin xyz=-1 0 0 rpy=0 0 0, axis 0 1 0, limit lower=-3.14159 upper=3.14159 effort=0.0 velocity=0.0
- added joint RightLeg_RightLowerLeg: type revolute, parent RightLeg, child RightLowerLeg, origin xyz=1 0 0 rpy=0 0 0, axis 0 1 0, limit lower=-3.14159 upper=3.14159 effort=0.0 velocity=0.0
- added joint Torso_LeftLeg: type revolute, parent Torso, child LeftLeg, origin xyz=-0.5 0 1 rpy=0 0 0, axis 0 1 0, limit lower=-3.14159 upper=3.14159 effort=0.0 velocity=0.0
- added joint Torso_RightLeg: type revolute, parent Torso, child RightLeg, origin xyz=0.5 0 1 rpy=0 0 0, axis 0 1 0, limit lower=-3.14159 upper=3.14159 effort=0.0 velocity=0.0
- joint Torso_BackLeg: axis 0 1 0 -> 1 0 0; origin xyz=2 0 1 rpy=0 0 0 -> xyz=0 -0.5 1 rpy=0 0 0
- joint Torso_FrontLeg: axis 0 1 0 -> 1 0 0; origin xyz=1 0 1 rpy=0 0 0 -> xyz=0 0.5 1 rpy=0 0 0

Commit message: new idea

File: body.urdf (robot description, URDF)
Before this commit: robot robot, 9 links, 8 joints
Links:
- link BackLeg: geometry collision box size=0.75 -0.2 0.2; visual box size=0.75 -0.2 0.2
- link BackLowerLeg: geometry collision box size=0.2 0.1 0.55; visual box size=0.2 0.1 0.55
- link FrontLeg: geometry collision box size=0.75 0.2 0.2; visual box size=0.75 0.2 0.2
- link FrontLowerLeg: geometry collision box size=0.2 0.1 0.55; visual box size=0.2 0.1 0.55
- link LeftLeg: geometry collision box size=0.75 0.2 0.2; visual box size=0.75 0.2 0.2
- link LeftLowerLeg: geometry collision box size=0.2 0.1 0.55; visual box size=0.2 0.1 0.55
- link RightLeg: geometry collision box size=0.75 -0.2 0.2; visual box size=0.75 -0.2 0.2
- link RightLowerLeg: geometry collision box size=0.2 0.1 0.55; visual box size=0.2 0.1 0.55
- link Torso: geometry collision box size=1 1.5 0.5; visual box size=1 1.5 0.5
Joints:
- joint BackLeg_BackLowerLeg: axis 1 0 0 -> 0 1 0; origin xyz=0 -1 0 rpy=0 0 0 -> xyz=-0.375 0 -0.2 rpy=0 0 0
- joint FrontLeg_FrontLowerLeg: axis 1 0 0 -> 0 1 0; origin xyz=0 1 0 rpy=0 0 0 -> xyz=0.375 0 -0.2 rpy=0 0 0
- joint LeftLeg_LeftLowerLeg: origin xyz=-1 0 0 rpy=0 0 0 -> xyz=-0.375 0 -0.2 rpy=0 0 0
- joint RightLeg_RightLowerLeg: origin xyz=1 0 0 rpy=0 0 0 -> xyz=0.375 0 -0.2 rpy=0 0 0
- joint Torso_BackLeg: axis 1 0 0 -> 0 1 0; origin xyz=0 -0.5 1 rpy=0 0 0 -> xyz=-0.5 -0.75 0.75 rpy=0 0 0
- joint Torso_FrontLeg: axis 1 0 0 -> 0 1 0; origin xyz=0 0.5 1 rpy=0 0 0 -> xyz=0.5 0.75 0.75 rpy=0 0 0
- joint Torso_LeftLeg: origin xyz=-0.5 0 1 rpy=0 0 0 -> xyz=-0.5 0.75 0.75 rpy=0 0 0
- joint Torso_RightLeg: origin xyz=0.5 0 1 rpy=0 0 0 -> xyz=0.5 -0.75 0.75 rpy=0 0 0

Commit message: stair climber

File: body.urdf (robot description, URDF)
Before this commit: robot robot, 9 links, 8 joints
Links:
- link BackLeg: geometry collision box size=0.3 -0.2 0.35; visual box size=0.3 -0.2 0.35
- link BackLowerLeg: geometry collision box size=0.25 0.1 0.44999999999999996; visual box size=0.25 0.1 0.44999999999999996
- link FrontLeg: geometry collision box size=0.3 0.2 0.35; visual box size=0.3 0.2 0.35
- link FrontLowerLeg: geometry collision box size=0.25 0.1 0.44999999999999996; visual box size=0.25 0.1 0.44999999999999996
- link LeftLeg: geometry collision box size=0.3 0.2 0.35; visual box size=0.3 0.2 0.35
- link LeftLowerLeg: geometry collision box size=0.25 0.1 0.44999999999999996; visual box size=0.25 0.1 0.44999999999999996
- link RightLeg: geometry collision box size=0.3 -0.2 0.35; visual box size=0.3 -0.2 0.35
- link RightLowerLeg: geometry collision box size=0.25 0.1 0.44999999999999996; visual box size=0.25 0.1 0.44999999999999996
- link Torso: geometry collision box size=1 0.7 0.4; visual box size=1 0.7 0.4
Joints:
- joint BackLeg_BackLowerLeg: origin xyz=-0.375 0 -0.2 rpy=0 0 0 -> xyz=-0.15 0 -0.35 rpy=0 0 0
- joint FrontLeg_FrontLowerLeg: origin xyz=0.375 0 -0.2 rpy=0 0 0 -> xyz=0.15 0 -0.35 rpy=0 0 0
- joint LeftLeg_LeftLowerLeg: origin xyz=-0.375 0 -0.2 rpy=0 0 0 -> xyz=-0.15 0 -0.35 rpy=0 0 0
- joint RightLeg_RightLowerLeg: origin xyz=0.375 0 -0.2 rpy=0 0 0 -> xyz=0.15 0 -0.35 rpy=0 0 0
- joint Torso_BackLeg: origin xyz=-0.5 -0.75 0.75 rpy=0 0 0 -> xyz=-0.5 -0.35 0.8 rpy=0 0 0
- joint Torso_FrontLeg: origin xyz=0.5 0.75 0.75 rpy=0 0 0 -> xyz=0.5 0.35 0.8 rpy=0 0 0
- joint Torso_LeftLeg: origin xyz=-0.5 0.75 0.75 rpy=0 0 0 -> xyz=-0.5 0.35 0.8 rpy=0 0 0
- joint Torso_RightLeg: origin xyz=0.5 -0.75 0.75 rpy=0 0 0 -> xyz=0.5 -0.35 0.8 rpy=0 0 0

Commit message: snake

File: body.urdf (robot description, URDF)
Before this commit: robot robot, 9 links, 8 joints
Links:
- removed link BackLeg
- removed link BackLowerLeg
- removed link FrontLeg
- removed link FrontLowerLeg
- removed link LeftLeg
- removed link LeftLowerLeg
- removed link RightLeg
- removed link RightLowerLeg
- removed link Torso
- added link 0, mass 1; collision box size=1.1797657967780515 0.2922351672983357 0.821599007946228; visual box size=1.1797657967780515 0.2922351672983357 0.821599007946228
- added link 1, mass 1; collision box size=0.3280788678207944 1.1598680642175943 0.2014567698136627; visual box size=0.3280788678207944 1.1598680642175943 0.2014567698136627
- added link 2, mass 1; collision box size=0.10591318504649579 0.6879822417076752 0.5468812245808187; visual box size=0.10591318504649579 0.6879822417076752 0.5468812245808187
- added link 3, mass 1; collision box size=0.35238462164824325 0.9925419877288727 0.44176093658392435; visual box size=0.35238462164824325 0.9925419877288727 0.44176093658392435
- added link 4, mass 1; collision box size=0.6364178012092112 1.0325377550558101 0.6947113235978345; visual box size=0.6364178012092112 1.0325377550558101 0.6947113235978345
- added link 5, mass 1; collision box size=0.4527570552091623 1.1246975744574115 0.6359802669981695; visual box size=0.4527570552091623 1.1246975744574115 0.6359802669981695
- added link 6, mass 1; collision box size=0.5435917298218795 0.6345200562743976 0.251639816647146; visual box size=0.5435917298218795 0.6345200562743976 0.251639816647146
Joints:
- removed joint BackLeg_BackLowerLeg
- removed joint FrontLeg_FrontLowerLeg
- removed joint LeftLeg_LeftLowerLeg
- removed joint RightLeg_RightLowerLeg
- removed joint Torso_BackLeg
- removed joint Torso_FrontLeg
- removed joint Torso_LeftLeg
- removed joint Torso_RightLeg
- added joint 0_1: type revolute, parent 0, child 1, origin xyz=0 0.2922351672983357 0.10072838490683135 rpy=0 0 0, axis 0 0 1, limit lower=-3.14159 upper=3.14159 effort=0.0 velocity=0.0
- added joint 1_2: type revolute, parent 1, child 2, origin xyz=0 1.1598680642175943 0.0 rpy=0 0 0, axis 0 0 1, limit lower=-3.14159 upper=3.14159 effort=0.0 velocity=0.0
- added joint 2_3: type revolute, parent 2, child 3, origin xyz=0 0.6879822417076752 0.12015208338513082 rpy=0 0 0, axis 0 0 1, limit lower=-3.14159 upper=3.14159 effort=0.0 velocity=0.0
- added joint 3_4: type revolute, parent 3, child 4, origin xyz=0 0.9925419877288727 0.0 rpy=0 0 0, axis 0 0 1, limit lower=-3.14159 upper=3.14159 effort=0.0 velocity=0.0
- added joint 4_5: type revolute, parent 4, child 5, origin xyz=0 1.0325377550558101 0.09710966520712255 rpy=0 0 0, axis 0 0 1, limit lower=-3.14159 upper=3.14159 effort=0.0 velocity=0.0
- added joint 5_6: type revolute, parent 5, child 6, origin xyz=0 1.1246975744574115 -0.19217022517551172 rpy=0 0 0, axis 0 0 1, limit lower=-3.14159 upper=3.14159 effort=0.0 velocity=0.0

Commit message: assign 7

File: body.urdf (robot description, URDF)
Before this commit: robot robot, 7 links, 6 joints
Links:
- removed link 1
- removed link 2
- removed link 3
- removed link 4
- removed link 5
- removed link 6
- added link 10, mass 1; collision box size=0.13805177806540894 0.3152825592344869 0.5476669085009627; visual box size=0.13805177806540894 0.3152825592344869 0.5476669085009627
- added link 11, mass 1; collision box size=0.13805177806540894 0.3152825592344869 0.5476669085009627; visual box size=0.13805177806540894 0.3152825592344869 0.5476669085009627
- added link 12, mass 1; collision box size=0.13805177806540894 0.3152825592344869 0.5476669085009627; visual box size=0.13805177806540894 0.3152825592344869 0.5476669085009627
- added link 13, mass 1; collision box size=0.13805177806540894 0.3152825592344869 0.5476669085009627; visual box size=0.13805177806540894 0.3152825592344869 0.5476669085009627
- added link 20, mass 1; collision box size=0.4035164851829698 0.11762477639901928 0.46540141505639865; visual box size=0.4035164851829698 0.11762477639901928 0.46540141505639865
- added link 21, mass 1; collision box size=0.4035164851829698 0.11762477639901928 0.46540141505639865; visual box size=0.4035164851829698 0.11762477639901928 0.46540141505639865
- added link 22, mass 1; collision box size=0.4035164851829698 0.11762477639901928 0.46540141505639865; visual box size=0.4035164851829698 0.11762477639901928 0.46540141505639865
- added link 23, mass 1; collision box size=0.4035164851829698 0.11762477639901928 0.46540141505639865; visual box size=0.4035164851829698 0.11762477639901928 0.46540141505639865
- added link 30, mass 1; collision box size=0.3400260798868108 0.16713472139286203 0.2293525939846727; visual box size=0.3400260798868108 0.16713472139286203 0.2293525939846727
- added link 31, mass 1; collision box size=0.3400260798868108 0.16713472139286203 0.2293525939846727; visual box size=0.3400260798868108 0.16713472139286203 0.2293525939846727
- added link 32, mass 1; collision box size=0.3400260798868108 0.16713472139286203 0.2293525939846727; visual box size=0.3400260798868108 0.16713472139286203 0.2293525939846727
- added link 33, mass 1; collision box size=0.3400260798868108 0.16713472139286203 0.2293525939846727; visual box size=0.3400260798868108 0.16713472139286203 0.2293525939846727
- added link 40, mass 1; collision box size=0.33630556950548407 0.25872942864360704 0.3512286703957769; visual box size=0.33630556950548407 0.25872942864360704 0.3512286703957769
- added link 41, mass 1; collision box size=0.33630556950548407 0.25872942864360704 0.3512286703957769; visual box size=0.33630556950548407 0.25872942864360704 0.3512286703957769
- added link 42, mass 1; collision box size=0.33630556950548407 0.25872942864360704 0.3512286703957769; visual box size=0.33630556950548407 0.25872942864360704 0.3512286703957769
- added link 43, mass 1; collision box size=0.33630556950548407 0.25872942864360704 0.3512286703957769; visual box size=0.33630556950548407 0.25872942864360704 0.3512286703957769
- added link 50, mass 1; collision box size=0.587802469441964 0.1548254862282004 0.3043294651455706; visual box size=0.587802469441964 0.1548254862282004 0.3043294651455706
- added link 51, mass 1; collision box size=0.587802469441964 0.1548254862282004 0.3043294651455706; visual box size=0.587802469441964 0.1548254862282004 0.3043294651455706
- added link 52, mass 1; collision box size=0.587802469441964 0.1548254862282004 0.3043294651455706; visual box size=0.587802469441964 0.1548254862282004 0.3043294651455706
- added link 53, mass 1; collision box size=0.587802469441964 0.1548254862282004 0.3043294651455706; visual box size=0.587802469441964 0.1548254862282004 0.3043294651455706
- link 0: geometry collision box size=1.0941111193739905 0.6539990997018729 0.38594162973688784; visual box size=1.0941111193739905 0.6539990997018729 0.38594162973688784
Joints:
- removed joint 0_1
- removed joint 1_2
- removed joint 2_3
- removed joint 3_4
- removed joint 4_5
- removed joint 5_6
- added joint 0_10: type revolute, parent 0, child 10, origin xyz=0.5470555596869953 0.32699954985093643 0.19297081486844392 rpy=0 0 0, axis 1 0 0, limit lower=-3.14159 upper=3.14159 effort=0.0 velocity=0.0
- added joint 0_11: type revolute, parent 0, child 11, origin xyz=-0.5470555596869953 0.32699954985093643 0.19297081486844392 rpy=0 0 0, axis 1 0 0, limit lower=-3.14159 upper=3.14159 effort=0.0 velocity=0.0
- added joint 0_12: type revolute, parent 0, child 12, origin xyz=0.5470555596869953 -0.32699954985093643 0.19297081486844392 rpy=0 0 0, axis 1 0 0, limit lower=-3.14159 upper=3.14159 effort=0.0 velocity=0.0
- added joint 0_13: type revolute, parent 0, child 13, origin xyz=-0.5470555596869953 -0.32699954985093643 0.19297081486844392 rpy=0 0 0, axis 1 0 0, limit lower=-3.14159 upper=3.14159 effort=0.0 velocity=0.0
- added joint 1_20: type revolute, parent 10, child 20, origin xyz=0 0.3152825592344869 0.039729892659755406 rpy=0 0 0, axis 1 0 0, limit lower=-3.14159 upper=3.14159 effort=0.0 velocity=0.0
- added joint 1_21: type revolute, parent 11, child 21, origin xyz=0 0.3152825592344869 0.039729892659755406 rpy=0 0 0, axis 1 0 0, limit lower=-3.14159 upper=3.14159 effort=0.0 velocity=0.0
- added joint 1_22: type revolute, parent 12, child 22, origin xyz=0 -0.3152825592344869 0.039729892659755406 rpy=0 0 0, axis 1 0 0, limit lower=-3.14159 upper=3.14159 effort=0.0 velocity=0.0
- added joint 1_23: type revolute, parent 13, child 23, origin xyz=0 -0.3152825592344869 0.039729892659755406 rpy=0 0 0, axis 1 0 0, limit lower=-3.14159 upper=3.14159 effort=0.0 velocity=0.0
- added joint 2_30: type revolute, parent 20, child 30, origin xyz=0 0.11762477639901928 -0.11802441053586298 rpy=0 0 0, axis 1 0 0, limit lower=-3.14159 upper=3.14159 effort=0.0 velocity=0.0
- added joint 2_31: type revolute, parent 21, child 31, origin xyz=0 0.11762477639901928 -0.11802441053586298 rpy=0 0 0, axis 1 0 0, limit lower=-3.14159 upper=3.14159 effort=0.0 velocity=0.0
- added joint 2_32: type revolute, parent 22, child 32, origin xyz=0 -0.11762477639901928 -0.11802441053586298 rpy=0 0 0, axis 1 0 0, limit lower=-3.14159 upper=3.14159 effort=0.0 velocity=0.0
- added joint 2_33: type revolute, parent 23, child 33, origin xyz=0 -0.11762477639901928 -0.11802441053586298 rpy=0 0 0, axis 1 0 0, limit lower=-3.14159 upper=3.14159 effort=0.0 velocity=0.0
- added joint 3_40: type revolute, parent 30, child 40, origin xyz=0 0.16713472139286203 0.0 rpy=0 0 0, axis 1 0 0, limit lower=-3.14159 upper=3.14159 effort=0.0 velocity=0.0
- added joint 3_41: type revolute, parent 31, child 41, origin xyz=0 0.16713472139286203 0.0 rpy=0 0 0, axis 1 0 0, limit lower=-3.14159 upper=3.14159 effort=0.0 velocity=0.0
- added joint 3_42: type revolute, parent 32, child 42, origin xyz=0 -0.16713472139286203 0.0 rpy=0 0 0, axis 1 0 0, limit lower=-3.14159 upper=3.14159 effort=0.0 velocity=0.0
- added joint 3_43: type revolute, parent 33, child 43, origin xyz=0 -0.16713472139286203 0.0 rpy=0 0 0, axis 1 0 0, limit lower=-3.14159 upper=3.14159 effort=0.0 velocity=0.0
- added joint 4_50: type revolute, parent 40, child 50, origin xyz=0 0.25872942864360704 0.03748843558044894 rpy=0 0 0, axis 1 0 0, limit lower=-3.14159 upper=3.14159 effort=0.0 velocity=0.0
- added joint 4_51: type revolute, parent 41, child 51, origin xyz=0 0.25872942864360704 0.03748843558044894 rpy=0 0 0, axis 1 0 0, limit lower=-3.14159 upper=3.14159 effort=0.0 velocity=0.0
- added joint 4_52: type revolute, parent 42, child 52, origin xyz=0 -0.25872942864360704 0.03748843558044894 rpy=0 0 0, axis 1 0 0, limit lower=-3.14159 upper=3.14159 effort=0.0 velocity=0.0
- added joint 4_53: type revolute, parent 43, child 53, origin xyz=0 -0.25872942864360704 0.03748843558044894 rpy=0 0 0, axis 1 0 0, limit lower=-3.14159 upper=3.14159 effort=0.0 velocity=0.0
